File: Espressylu-0.6.sch (EAGLE design)
At the start: 135 parts, among them J1 4P-TERM-BLOCK284391-4, J10 MICROSD, J11 2x7, J2 M02POLAR, J3 M02POLAR, J4 USB-MICRO-PTH, J5 M02POLAR, J6 HOTEND-1, J7 HOTBED, J8 M02POLAR, J9 M02POLAR, P1 POLOLU-X, P2 POLOLU-Y, P3 POLOLU-Z, P4 POLOLU-E1, Q1 PMV45EN, Q2 PSMN1R8-40YLC, Q3 MMUN2211LT3G, Q4 PSMN1R8-40YLC, U1 DRTR5V0U2SR, U2 MCP1402T, U3 LMR16006X, U4 L78L15ABUTR, U5 MCP1402T, X1 12MHZ

Commit message: Layout cleanup
Moved the stepper motor headers closer to the connectors. Cleaned up the
schematic and labels.
Parts:
- C10: value 4.7uF -> 0.1uF; device teensylu:CAPACITOR_0603 -> teensylu:CAPACITOR_0402; MANUFACTURER_PART_NUMBER CL10B475KQ8NQNC -> CL05A104KQ5NNNC
- C11: MANUFACTURER (none) -> Samsung; MANUFACTURER_PART_NUMBER (none) -> CL05A104KQ5NNNC; TOLERANCE 20% -> 10%; VDC 50V -> 6.3V
- C15: MANUFACTURER Murata -> Samsung; MANUFACTURER_PART_NUMBER GRM188R71C104KA01D -> CL05A104KQ5NNNC; VDC 16V -> 6.3V
- C20: value 0.1uF -> 4.7uF; device teensylu:CAPACITOR_0402 -> teensylu:CAPACITOR_1206; MANUFACTURER Samsung -> Yaiyo Yuden; MANUFACTURER_PART_NUMBER CL05A104KQ5NNNC -> UMK316AB7475KL-T; VDC 6.3V -> 50v
- C21: value 0.1uF -> 4.7uF; device teensylu:CAPACITOR_0402 -> teensylu:CAPACITOR_0603; MANUFACTURER_PART_NUMBER CL05A104KQ5NNNC -> CL10B475KQ8NQNC
- C23: value 4.7uF -> 0.1uF; device teensylu:CAPACITOR_0603 -> teensylu:CAPACITOR_0402; MANUFACTURER Samsung -> (none); MANUFACTURER_PART_NUMBER CL10B475KQ8NQNC -> (none); TOLERANCE 10% -> 20%; VDC 6.3V -> 50V
- C27: value 0.1uF -> 10pF; MANUFACTURER_PART_NUMBER CL05A104KQ5NNNC -> CL10C100JB8NCNC; TOLERANCE 10% -> 5%; VDC 6.3V -> 50V
- C29: value 10pF -> 100uF; device teensylu:CAPACITOR_0402 -> teensylu:CPOL-USD; MANUFACTURER Samsung -> Panasonic; MANUFACTURER_PART_NUMBER CL10C100JB8NCNC -> EEE-FTH101XAP; TOLERANCE 5% -> 20%; VDC 50V -> 50v
- C31: value 100uF -> 0.1uF; device teensylu:CPOL-USD -> teensylu:CAPACITOR_0402; MANUFACTURER Panasonic -> (none); MANUFACTURER_PART_NUMBER EEE-FTH101XAP -> (none); VDC 50v -> 50V
- C33: value 0.1uF -> 1uF
- C34: value 1uF -> 15pF; MANUFACTURER (none) -> Samsung; MANUFACTURER_PART_NUMBER (none) -> CL05C150JB5NNNC; TOLERANCE 20% -> 5%
- C35: value 0.1uF -> 15pF; MANUFACTURER (none) -> Samsung; MANUFACTURER_PART_NUMBER (none) -> CL05C150JB5NNNC; TOLERANCE 20% -> 5%
- C36: value 15pF -> 0.1uF; MANUFACTURER Samsung -> (none); MANUFACTURER_PART_NUMBER CL05C150JB5NNNC -> (none); TOLERANCE 5% -> 20%
- C37: value 15pF -> 100uF; device teensylu:CAPACITOR_0402 -> teensylu:CPOL-USD; MANUFACTURER Samsung -> Panasonic; MANUFACTURER_PART_NUMBER CL05C150JB5NNNC -> EEE-FTH101XAP; TOLERANCE 5% -> 20%; VDC 50V -> 50v
- C38: value 10uF -> 4.7uF; device teensylu:CAPACITOR_0402 -> teensylu:CAPACITOR_0603; MANUFACTURER Murata -> Samsung; MANUFACTURER_PART_NUMBER GRM188R61C106MA73D -> CL10B475KQ8NQNC; TOLERANCE 20% -> 10%; VDC 16V -> 6.3V
- C40: value 100uF -> 10uF; device teensylu:CPOL-USD -> teensylu:CAPACITOR_0402; MANUFACTURER Panasonic -> Murata; MANUFACTURER_PART_NUMBER EEE-FTH101XAP -> GRM188R61C106MA73D; VDC 50v -> 16V
- C41: value 100uF -> 0.1uF; device teensylu:CPOL-USD -> teensylu:CAPACITOR_0402; MANUFACTURER Panasonic -> Murata; MANUFACTURER_PART_NUMBER EEE-FTH101XAP -> GRM188R71C104KA01D; TOLERANCE 20% -> 10%; VDC 50v -> 16V
- C45: value 4.7uF -> 100uF; device teensylu:CAPACITOR_0603 -> teensylu:CPOL-USD; MANUFACTURER Samsung -> Panasonic; MANUFACTURER_PART_NUMBER CL10B475KQ8NQNC -> EEE-FTH101XAP; TOLERANCE 10% -> 20%; VDC 6.3V -> 50v
- C9: device teensylu:CAPACITOR_1206 -> teensylu:CAPACITOR_0603; MANUFACTURER Yaiyo Yuden -> Samsung; MANUFACTURER_PART_NUMBER UMK316AB7475KL-T -> CL10B475KQ8NQNC; VDC 50v -> 6.3V
- J10: value MICROSD -> M02POLAR; device teensylu:MICROSD -> teensylu:M02POLAR; DESCRIPTION CONN MICRO SD CARD PUSH-PULL R/A -> CONN HEADER 2POS .100 VERT TIN; MANUFACTURER (none) -> Molex; MANUFACTURER_PART_NUMBER (none) -> 0022272021; NOTES (none) -> Can use alternative part for Right Angle. MFG: TE Connectiv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
- J11: value 2x7 -> M02POLAR; device teensylu:JP7Q -> teensylu:M02POLAR; DESCRIPTION DIL VERTICAL PC TAIL PIN HEADER -> CONN HEADER 2POS .100 VERT TIN; MANUFACTURER Harwin -> Molex; MANUFACTURER_PART_NUMBER M20-9980746 -> 0022272021; NOTES (none) -> Can use alternative part for Right Angle. MFG: TE Connectiv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
- J4: value USB-MICRO-PTH -> M02POLAR; device teensylu:USB-MICRO-PTH -> teensylu:M02POLAR; DESCRIPTION (none) -> CONN HEADER 2POS .100 VERT TIN; MANUFACTURER (none) -> Molex; MANUFACTURER_PART_NUMBER (none) -> 0022272021; NOTES (none) -> Can use alternative part for Right Angle. MFG: TE Connectiv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
- J5: value M02POLAR -> HOTEND-1; device teensylu:M02POLAR -> teensylu:4P-TERM-BLOCK284391-4; DESCRIPTION CONN HEADER 2POS .100 VERT TIN -> (none); MANUFACTURER Molex -> (none); MANUFACTURER_PART_NUMBER 0022272021 -> (none); NOTES Can use alternative part for Right Angle. MFG: TE Connectiv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 -> (none)
- J6: value HOTEND-1 -> 2x7; device teensylu:4P-TERM-BLOCK284391-4 -> teensylu:JP7Q; DESCRIPTION (none) -> DIL VERTICAL PC TAIL PIN HEADER; MANUFACTURER (none) -> Harwin; MANUFACTURER_PART_NUMBER (none) -> M20-9980746
- J8: value M02POLAR -> MICROSD; device teensylu:M02POLAR -> teensylu:MICROSD; DESCRIPTION CONN HEADER 2POS .100 VERT TIN -> CONN MICRO SD CARD PUSH-PULL R/A; MANUFACTURER Molex -> (none); MANUFACTURER_PART_NUMBER 0022272021 -> (none); NOTES Can use alternative part for Right Angle. MFG: TE Connectiv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 -> (none)
- J9: value M02POLAR -> USB-MICRO-PTH; device teensylu:M02POLAR -> teensylu:USB-MICRO-PTH; DESCRIPTION CONN HEADER 2POS .100 VERT TIN -> (none); MANUFACTURER Molex -> (none); MANUFACTURER_PART_NUMBER 0022272021 -> (none); NOTES Can use alternative part for Right Angle. MFG: TE Connectiv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 -> (none)
- JP10: value MOT-Y -> M03POLAR; device teensylu:M04POLAR -> teensylu:M03POLAR; DESCRIPTION (none) -> CONN HEADER 3POS .100 VERT TIN; MANUFACTURER (none) -> Molex; MANUFACTURER_PART_NUMBER (none) -> 0022272031; NOTES Can use alternative part for Right Angle. MFG: TE Connectivity PN: 640455-4 -> Can use alternative part for Right Angle. MFG: TE Connectivity PN: 640455-3
- JP11: value MOT-E1 -> MOT-X
- JP12: value MOT-Z -> MOT-Y
- JP13: value JTAG-HEADER -> MOT-E1; device teensylu:JTAG-HEADER -> teensylu:M04POLAR; NOTES (none) -> Can use alternative part for Right Angle. MFG: TE Connectiv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
- JP14: value ISP -> MOT-Z; device teensylu:PROGHEADER -> teensylu:M04POLAR; NOTES (none) -> Can use alternative part for Right Angle. MFG: TE Connectiv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
- JP4: value JUMPER-3PTH -> JTAG-HEADER; device teensylu:JUMPER-3PTH -> teensylu:JTAG-HEADER
- JP5: value Z-STOP -> ISP; device teensylu:M04POLAR -> teensylu:PROGHEADER; NOTES Can use alternative part for Right Angle. MFG: TE Connectiv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 -> (none)
- JP6: value M03POLAR -> JUMPER-3PTH; device teensylu:M03POLAR -> teensylu:JUMPER-3PTH; DESCRIPTION CONN HEADER 3POS .100 VERT TIN -> (none); MANUFACTURER Molex -> (none); MANUFACTURER_PART_NUMBER 0022272031 -> (none); NOTES Can use alternative part for Right Angle. MFG: TE Connectiv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 -> (none)
- JP7: value M03POLAR -> Z-STOP; device teensylu:M03POLAR -> teensylu:M04POLAR; DESCRIPTION CONN HEADER 3POS .100 VERT TIN -> (none); MANUFACTURER Molex -> (none); MANUFACTURER_PART_NUMBER 0022272031 -> (none); NOTES Can use alternative part for Right Angle. MFG: TE Connectivity PN: 640455-3 -> Can use alternative part for Right Angle. MFG: TE Connectivity PN: 640455-4
- JP9: value MOT-X -> M03POLAR; device teensylu:M04POLAR -> teensylu:M03POLAR; DESCRIPTION (none) -> CONN HEADER 3POS .100 VERT TIN; MANUFACTURER (none) -> Molex; MANUFACTURER_PART_NUMBER (none) -> 0022272031; NOTES Can use alternative part for Right Angle. MFG: TE Connectivity PN: 640455-4 -> Can use alternative part for Right Angle. MFG: TE Connectivity PN: 640455-3
- Q3: value MMUN2211LT3G -> PSMN1R8-40YLC; device teensylu:TRANSISTOR_NPN_BIASSOT23C -> teensylu:PSMN1R8-40YLCPOWERPACK-S08; DESCRIPTION TRANS PREBIAS NPN 246MW SOT23-3 -> (none); MANUFACTURER ON Semiconductor -> (none); MANUFACTURER_PART_NUMBER MMUN2211LT3G -> (none)
- Q4: value PSMN1R8-40YLC -> MMUN2211LT3G; device teensylu:PSMN1R8-40YLCPOWERPACK-S08 -> teensylu:TRANSISTOR_NPN_BIASSOT23C; DESCRIPTION (none) -> TRANS PREBIAS NPN 246MW SOT23-3; MANUFACTURER (none) -> ON Semiconductor; MANUFACTURER_PART_NUMBER (none) -> MMUN2211LT3G
- R10: value 6.8k -> 39
- R11: value 100k -> 39; TOLERANCE (none) -> 1%
- R12: value 39 -> 0; TOLERANCE 1% -> (none)
- R13: value 39 -> 28k
- R14: value 0 -> 8.45k; TOLERANCE (none) -> 1%
- R4: value 15k -> 10k
- R5: value 10k -> 15k
- R8: value 28k -> 6.8k
- R9: value 8.45k -> 100k; TOLERANCE 1% -> (none)
- U1: value DRTR5V0U2SR -> MCP1402T; device teensylu:DRTR5V0U2SR -> teensylu:MCP1402T
- U2: value MCP1402T -> LMR16006X; device teensylu:MCP1402T -> teensylu:LMR16006X
- U3: value LMR16006X -> MCP1402T; device teensylu:LMR16006X -> teensylu:MCP1402T
- U5: value MCP1402T -> (none); device teensylu:MCP1402T -> teensylu:ATSAM3A8C-LQFP100
- U6: value (none) -> DRTR5V0U2SR; device teensylu:ATSAM3A8C-LQFP100 -> teensylu:DRTR5V0U2SR
Connections:
- net !E1-ENABLE: now also U5G$2.PB23/CTS2.SPI0_NPCS3/WKUP14; no longer U6G$2.PB23/CTS2.SPI0_NPCS3/WKUP14
- net !HOTBED: now also U3.IN, U5G$1.PA5/TIOA2/PWMFI0/WKUP2; no longer U5.IN, U6G$1.PA5/TIOA2/PWMFI0/WKUP2
- net !HOTEND-1: now also R4.1, U1.IN, U5G$1.PA1/CANRX0/PCK0/WKUP0; no longer R5.1, U2.IN, U6G$1.PA1/CANRX0/PCK0/WKUP0
- net !PWM-FAN: now also U5G$2.PB5/TIOB5; no longer U6G$2.PB5/TIOB5
- net !RESET: now also JP4.10, JP5.2, U5G$3.!NRST; no longer JP13.10, JP14.2, U6G$3.!NRST
- net !X-ENABLE: now also U5G$1.PA14/RTS1/TK; no longer U6G$1.PA14/RTS1/TK
- net !Y-ENABLE: now also U5G$1.PA11/TXD0/ADTRG/WKUP6; no longer U6G$1.PA11/TXD0/ADTRG/WKUP6
- net !Z-ENABLE: now also U5G$2.PB26/CTS0/TCLK0/WKUP15; no longer U6G$2.PB26/CTS0/TCLK0/WKUP15
- net +15V: now also C23.1, C31.1, C36.1, U1.VDD, U3.VDD; no longer C11.1, C33.1, C35.1, U2.VDD, U5.VDD
- net +3V3: now also C13.1, C15.1, C17.1, C26.1, C38.1, C9.1, J6.2, J8.VDD, JP4.1, JP5.5, JP6.3, JP7.2, R13.1, R9.2, U5G$3.VDDBU, U5G$3.VDDIN, U5G$3.VDDIO1, U5G$3.VDDIO2, U5G$3.VDDIO3; no longer C10.1, C18.1, C20.1, C22.1, C27.1, C45.1, J10.VDD, J11.2, JP13.1, JP14.5, JP4.3, JP5.2, R11.2, R8.1, U6G$3.VDDBU, U6G$3.VDDIN, U6G$3.VDDIO1, U6G$3.VDDIO2, U6G$3.VDDIO3
- net 24V: now also C20.1, C29.+, C33.1, C37.+, C45.+, J4.1, J5.3, J5.4, JP6.1, JP7.4, R5.1, U2.VIN; no longer C31.+, C34.1, C40.+, C41.+, C9.1, J11.3, J5.1, J6.4, JP4.1, JP5.4, R4.1, U3.VIN
- net 5VREG_CB: now also U2.CB; no longer U3.CB
- net 5VREG_FB: now also R13.2, R14.1, U2.FB; no longer R8.2, R9.1, U3.FB
- net 5VREG_SW: now also U2.SW; no longer U3.SW
- net AD3: now also J6.13, U5G$1.PA6/TIOB2/NCS0/AD3; no longer J11.13, U6G$1.PA6/TIOB2/NCS0/AD3
- net ADVREF: now also C25.1, U5G$3.ADVREF; no longer C26.1, U6G$3.ADVREF
- net B-THERM: now also C40.2, J11.1, U5G$2.PB20/TXD2/SPI0_NPCS1/AD13; no longer C39.2, J9.1, U6G$2.PB20/TXD2/SPI0_NPCS1/AD13
- net E-MOT-1A: now also JP13.3; no longer JP11.3
- net E-MOT-1B: now also JP13.4; no longer JP11.4
- net E-MOT-2A: now also JP13.2; no longer JP11.2
- net E-MOT-2B: now also JP13.1; no longer JP11.1
- net E-STOP: now also JP10.1, U5G$2.PB16/TCLK5/PWML0/DAC1; no longer JP8.1, U6G$2.PB16/TCLK5/PWML0/DAC1
- net E1-DIR: now also U5G$2.PB14/CANTX1/PWMH2; no longer U6G$2.PB14/CANTX1/PWMH2
- net E1-STEP: now also U5G$2.PB22/RTS2/PCK0; no longer U6G$2.PB22/RTS2/PCK0
- net E1-THERM: now also C39.2, J10.1, U5G$2.PB21/RXD2.SPI0_NPCS2/AD14; no longer C38.2, J8.1, U6G$2.PB21/RXD2.SPI0_NPCS2/AD14
- net ENDSTOP+V: now also JP10.2, JP9.2; no longer JP4.2, JP7.2
- net ERASE: now also U5G$3.PC0/ERASE; no longer U6G$3.PC0/ERASE
- net GND: now also C15.2, C29.-, C31.2, C34.1, C35.1, C36.2, C37.-, C38.2, C40.1, C41.1, C45.-, J10.2, J11.2, J6.1, J8.CD1, J8.GND, J8.SHEILD@1, J8.SHIELD@2, J8.SHIELD@3, J8.SHIELD@4, J9.GND, JP10.3, JP4.3, JP4.5, JP4.9, JP5.1, JP9.3, Q3.S1, Q3.S2, Q3.S3, Q4.E, R12.2, R4.2, R8.1, U1.GND1, U1.GND2, U2.GND, U3.GND1, U3.GND2, U5G$3.GND1, U5G$3.GND2, U5G$3.GND3, U5G$3.GND4, U5G$3.GND5, U5G$3.GNDANA, U5G$3.GNDPLL, U5G$3.GNDUTMI, U5G$3.JTAGSEL, U6.GND; no longer C15.1, C29.2, C31.-, C34.2, C35.2, C36.1, C37.1, C38.1, C40.-, C41.-, C45.2, J10.CD1, J10.GND, J10.SHEILD@1, J10.SHIELD@2, J10.SHIELD@3, J10.SHIELD@4, J11.1, J4.GND, J8.2, J9.2, JP13.3, JP13.5, JP13.9, JP14.1, JP5.3, JP6.3, Q3.E, Q4.S1, Q4.S2, Q4.S3, R10.1, R5.2, R9.2, U1.GND, U2.GND1, U2.GND2, U3.GND, U5.GND1, U5.GND2, U6G$3.GND1, U6G$3.GND2, U6G$3.GND3, U6G$3.GND4, U6G$3.GND5, U6G$3.GNDANA, U6G$3.GNDPLL, U6G$3.GNDUTMI, U6G$3.JTAGSEL
- net HOTBED-GND: now also Q3.D; no longer Q4.D
- net HOTEND-GND: now also J5.1, J5.2; no longer J6.1, J6.2
- net JTAG_TCK: now also JP4.4, U5G$2.PB28/TCK/SWCLK; no longer JP13.4, U6G$2.PB28/TCK/SWCLK
- net JTAG_TDI: now also JP4.8, U5G$2.PB29/TDI; no longer JP13.8, U6G$2.PB29/TDI
- net JTAG_TDO: now also JP4.6, U5G$2.PB30/TDO/TRACESWO; no longer JP13.6, U6G$2.PB30/TDO/TRACESWO
- net JTAG_TMS: now also JP4.2, U5G$2.PB31/TMS/SWDIO; no longer JP13.2, U6G$2.PB31/TMS/SWDIO
- net MCCDA: now also J8.CMD/DI, U5G$1.PA20/MCCDA/PWML2; no longer J10.CMD/DI, U6G$1.PA20/MCCDA/PWML2
- net MCCK: now also J8.CLK, U5G$1.PA19/MCCK/PWMH1; no longer J10.CLK, U6G$1.PA19/MCCK/PWMH1
- net MCDA0: now also J8.DAT0/DO, U5G$1.PA21/MCDA0/PWML0; no longer J10.DAT0/DO, U6G$1.PA21/MCDA0/PWML0
- net MCDA1: now also J8.DAT1, U5G$1.PA22/MCDA1/TCLK3/AD4; no longer J10.DAT1, U6G$1.PA22/MCDA1/TCLK3/AD4
- net MCDA2: now also J8.DAT2, U5G$1.PA23/MCDA2/TCLK4/AD5; no longer J10.DAT2, U6G$1.PA23/MCDA2/TCLK4/AD5
- net MCDA3: now also J8.DAT3/CS, U5G$1.PA24/MCDA3/PCK1/AD6; no longer J10.DAT3/CS, U6G$1.PA24/MCDA3/PCK1/AD6
- net MISO: now also JP5.6, U5G$1.PA25/SPI0_MISO/A18; no longer JP14.6, U6G$1.PA25/SPI0_MISO/A18
- net MOSI: now also JP5.3, U5G$1.PA26/SPI0_MOSI/A19; no longer JP14.3, U6G$1.PA26/SPI0_MOSI/A19
- net N$12: now also R11.2, U5G$3.DFSDP; no longer R13.2, U6G$3.DFSDP
- net N$14: now also U3.OUT; no longer U5.OUT
- net N$15: now also U1.OUT; no longer U2.OUT
- net N$2: now also Q3.G; no longer Q4.G
- net N$3: now also R5.2, U2.!SHDN; no longer R4.2, U3.!SHDN
- net N$4: now also R9.1, U5G$3.FWUP; no longer R11.1, U6G$3.FWUP
- net N$5: now also J4.2; no longer J5.2
- net N$7: now also R12.1, U5G$3.TST; no longer R14.1, U6G$3.TST
- net N$9: now also R10.2, U5G$3.DFSDM; no longer R12.2, U6G$3.DFSDM
- net PA15: now also U5G$1.PA15/CTS1/TF/WKUP8; no longer U6G$1.PA15/CTS1/TF/WKUP8
- net PA17: now also U5G$1.PA17/TWD0/SPCK0; no longer U6G$1.PA17/TWD0/SPCK0
- net PA2: now also J6.12, U5G$1.PA2/TIOA1/NANDRDY/AD0; no longer J11.12, U6G$1.PA2/TIOA1/NANDRDY/AD0
- net PA28: now also J6.5, U5G$1.PA28/SPI0_NPCS0/PCK2/WKUP11; no longer J11.5, U6G$1.PA28/SPI0_NPCS0/PCK2/WKUP11
- net PA29: now also J6.4, U5G$1.PA29/SPI0_NPCS1/NRD; no longer J11.4, U6G$1.PA29/SPI0_NPCS1/NRD
- net PA3: now also J6.11, U5G$1.PA3/TIOB1/PWMFI0/WKUP1; no longer J11.11, U6G$1.PA3/TIOB1/PWMFI0/WKUP1
- net PA4: now also J6.14, U5G$1.PA4/TCLK1/NWAIT/AD2; no longer J11.14, U6G$1.PA4/TCLK1/NWAIT/AD2
- net PB12: now also J6.9, U5G$2.PB12/TWD1/PWMH0/AD8; no longer J11.9, U6G$2.PB12/TWD1/PWMH0/AD8
- net PB13: now also J6.10, U5G$2.PB13/TWCK1/PWMH1/AD9; no longer J11.10, U6G$2.PB13/TWCK1/PWMH1/AD9
- net PB17: now also J6.8, U5G$2.PB17/RF/PWML1/AD10; no longer J11.8, U6G$2.PB17/RF/PWML1/AD10
- net PB18: now also J6.6, U5G$2.PB18/RD/PWML2/AD11; no longer J11.6, U6G$2.PB18/RD/PWML2/AD11
- net PB19: now also J6.7, U5G$2.PB19/RK/PWML3/AD12; no longer J11.7, U6G$2.PB19/RK/PWML3/AD12
- net SCLK: now also JP5.4, U5G$1.PA27/SPI0_SPCK/A20/WKUP10; no longer JP14.4, U6G$1.PA27/SPI0_SPCK/A20/WKUP10
- net SDCD: now also J8.CD2, U5G$1.PA18/TWCK0/A20/WKUP9; no longer J10.CD2, U6G$1.PA18/TWCK0/A20/WKUP9
- net USB_DN: now also J9.D-, R10.1, U5G$3.DHSDM, U6.IO2; no longer J4.D-, R12.1, U1.IO2, U6G$3.DHSDM
- net USB_DP: now also J9.D+, R11.1, U5G$3.DHSDP, U6.IO1; no longer J4.D+, R13.1, U1.IO1, U6G$3.DHSDP
- net VBG: now also C27.1, R8.2, U5G$3.VBG; no longer C29.1, R10.2, U6G$3.VBG
- net VBUS: now also C41.2, J9.VBUS, U5G$3.VBUS, U6.VCC; no longer C15.2, J4.VBUS, U1.VCC, U6G$3.VBUS
- net VDD: now also C12.1, C18.1, C22.1, U5G$3.VDDCORE1, U5G$3.VDDCORE2, U5G$3.VDDCORE3, U5G$3.VDDCORE4, U5G$3.VDDCORE5, U5G$3.VDDOUT; no longer C17.1, C21.1, C24.1, U6G$3.VDDCORE1, U6G$3.VDDCORE2, U6G$3.VDDCORE3, U6G$3.VDDCORE4, U6G$3.VDDCORE5, U6G$3.VDDOUT
- net VDDANA: now also C10.1, U5G$3.VDDANA; no longer C12.1, U6G$3.VDDANA
- net VDDPLL: now also C11.1, U5G$3.VDDPLL; no longer C13.1, U6G$3.VDDPLL
- net VDDUTMI: now also C21.1, C24.1, U5G$3.VDDUTMI; no longer C23.1, C25.1, U6G$3.VDDUTMI
- net X-DIR: now also U5G$1.PA12/RXD1/PWML1/WKUP7; no longer U6G$1.PA12/RXD1/PWML1/WKUP7
- net X-MOT-1A: now also JP11.3; no longer JP9.3
- net X-MOT-1B: now also JP11.4; no longer JP9.4
- net X-MOT-2A: now also JP11.2; no longer JP9.2
- net X-MOT-2B: now also JP11.1; no longer JP9.1
- net X-STEP: now also U5G$1.PA13/TXD1/PWMH2; no longer U6G$1.PA13/TXD1/PWMH2
- net X-STOP: now also JP8.1, U5G$2.PB15/CANRX1/PWMH3/DAC0; no longer JP6.1, U6G$2.PB15/CANRX1/PWMH3/DAC0
- net XTAL1: now also C35.2, U5G$3.XIN; no longer C37.2, U6G$3.XIN
- net XTAL2: now also C34.2, U5G$3.XOUT; no longer C36.2, U6G$3.XOUT
- net Y-DIR: now also U5G$1.PA9/UTXD/PWMH3; no longer U6G$1.PA9/UTXD/PWMH3
- net Y-MOT-1A: now also JP12.3; no longer JP10.3
- net Y-MOT-1B: now also JP12.4; no longer JP10.4
- net Y-MOT-2A: now also JP12.2; no longer JP10.2
- net Y-MOT-2B: now also JP12.1; no longer JP10.1
- net Y-STEP: now also U5G$1.PA10/RXD0/DATRG/WKUP5; no longer U6G$1.PA10/RXD0/DATRG/WKUP5
- net Y-STOP: now also JP9.1, U5G$1.PA7/TCLK2/NCS1/WKUP3; no longer JP7.1, U6G$1.PA7/TCLK2/NCS1/WKUP3
- net Z-DIR: now also U5G$2.PB24/SCK2/NCS2; no longer U6G$2.PB24/SCK2/NCS2
- net Z-MOT-1A: now also JP14.3; no longer JP12.3
- net Z-MOT-1B: now also JP14.4; no longer JP12.4
- net Z-MOT-2A: now also JP14.2; no longer JP12.2
- net Z-MOT-2B: now also JP14.1; no longer JP12.1
- net Z-STEP: now also U5G$2.PB25/RTS0/TIOA0; no longer U6G$2.PB25/RTS0/TIOA0
- net Z-STOP: now also Q4.C, U5G$1.PA8/URXD/PWMH0/WKUP4; no longer Q3.C, U6G$1.PA8/URXD/PWMH0/WKUP4
- net Z-STOP-BIAS: now also JP7.1, Q4.B; no longer JP5.1, Q3.B
Other:
- note added: "15v supply for mosfet drivers"
- note added: "3.3v Switching Regulator"
- note added: "Espressylu"
- note added: "Rev 0.6"
- note removed: "5v Switching Regulator"
- note removed: "Extension Pin Headers"
- note removed: "Rev 1.3a"
- note removed: "TeensyluV1"
- moved on the sheet: C10, C11, C12, C13, C14, C15, C16, C17, C18, C19, C20, C21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
