File: Espressylu-0.7.sch (EAGLE design)
At the start: 135 parts, among them J1 4P-TERM-BLOCK284391-4, J10 M02POLAR, J11 M02POLAR, J2 M02POLAR, J3 M02POLAR, J4 M02POLAR, J5 HOTEND-1, J6 2x7, J7 HOTBED, J8 MICROSD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

Commit message: Cleaned up Silkscreen and added caps
I cleaned up the silkscreen for all of the components.
Capacitors were added to the motor driver VCC pins.
More GND Vias were added to reduce noise.
The mosfets were shifted away from the connectors slightly.
The stepper motor connectors were shifted slightly closer to the edge of
the board.
All of the HV pins are labelled as 24v. This board should only be used
with 24v.
Parts:
- added C46, C47, C48, C49: 100uF, teensylu:CPOL-USD
- C42, C43, C44, C45: value 100uF -> 4.7uF; device teensylu:CPOL-USD -> teensylu:CAPACITOR_0603; MANUFACTURER Panasonic -> Samsung; MANUFACTURER_PART_NUMBER EEE-FTH101XAP -> CL10B475KQ8NQNC; TOLERANCE 20% -> 10%; VDC 50v -> 6.3V
- S1: value (none) -> RESET; device teensylu:TAC_SWITCH_2P-SMD -> teensylu:TAC_SWITCH_4P4P-SMD
- S2: value (none) -> ERASE; device teensylu:TAC_SWITCH_2P-SMD -> teensylu:TAC_SWITCH_4P4P-SMD
Connections:
- net +3V3: now also C42.2, C43.2, C44.2, C45.2, S2.3; no longer S2.2
- net 24V: now also C46.+, C47.+, C48.+, C49.+; no longer C42.+, C43.+, C44.+, C45.+
- net GND: now also C42.1, C43.1, C44.1, C45.1, C46.-, C47.-, C48.-, C49.-, S1.3, S1.4; no longer C42.-, C43.-, C44.-, C45.-, S1.2
Other:
- note added: "Rev 0.7"
- note removed: "Rev 0.6"
